Commit message: feat: fixing non-unique link names

File: clover_description/urdf/sensors/distance_sensor.urdf.xacro (robot description, xacro)
@@ -5,11 +5,11 @@
   <xacro:include filename="../camera_sensor.urdf.xacro"/>
   <xacro:macro name="distance_sensor" params="name:=lidar_VL53L4CX index parent x:=0 y:=0 z:=0 roll:=0 pitch:=0 yaw:=0 range_min range_max resolution:=0.01 rate:=10 fov:=0.3141593">
-    <joint name="${name}_joint" type="fixed">
+    <joint name="${name}_${index}_joint" type="fixed">
       <origin xyz="${x} ${y} ${z}"
               rpy="${roll} ${pitch} ${yaw}"/>
       <parent link="${parent}"/>
-      <child link="${name}_link"/>
+      <child link="${name}_${index}_link"/>
     </joint>
-    <link name="${name}_link">
+    <link name="${name}_${index}_link">
       <visual>
         <origin xyz="0 0 0" rpy="0 0 0"/>
@@ -30,10 +30,10 @@
       </inertial>
     </link>
-    <gazebo reference="${name}_joint">
+    <gazebo reference="${name}_${index}_joint">
       <disableFixedJointLumping>true</disableFixedJointLumping>
       <preserveFixedJoint>true</preserveFixedJoint>
     </gazebo>
-    <gazebo reference="${name}_link">
-      <sensor type="ray" name="${name}">
+    <gazebo reference="${name}_${index}_link">
+      <sensor type="ray" name="${name}_${index}">
         <pose>0 0 0 0 0 0</pose>
         <ray>

Commit message: fix: sensor size and healthcheck disabling

File: clover_description/urdf/sensors/distance_sensor.urdf.xacro (robot description, xacro)
@@ -14,5 +14,5 @@
         <origin xyz="0 0 0" rpy="0 0 0"/>
         <geometry>
-          <box size="0.001 0.005 0.005"/>
+          <box size="0.0015 0.0175 0.025"/> <!-- dimension of Adafruit VL53L4CX -->
         </geometry>
       </visual>

Commit message: fix: sensors geometry

File: clover_description/urdf/sensors/distance_sensor.urdf.xacro (robot description, xacro)
@@ -14,5 +14,5 @@
         <origin xyz="0 0 0" rpy="0 0 0"/>
         <geometry>
-          <box size="0.0015 0.0175 0.025"/> <!-- dimension of Adafruit VL53L4CX -->
+          <box size="0.0015 0.025 0.0175"/> <!-- dimension of Adafruit VL53L4CX -->
         </geometry>
       </visual>
@@ -20,9 +20,9 @@
         <origin xyz="0 0 0" rpy="0 0 0"/>
         <geometry>
-          <box size="0.001 0.001 0.005"/>
+          <box size="0.0015 0.025 0.0175"/> <!-- dimension of Adafruit VL53L4CX -->
         </geometry>
       </collision>
       <inertial>
-        <mass value="0.015"/>
+        <mass value="0.001"/>
         <origin xyz="0 0 0"/>
         <inertia ixx="4.15e-6" iyy="2.407e-6" izz="2.407e-6" ixy="0" ixz="0" iyz="0"/>

Commit message: fix: removing collision parameters to allow for min range

File: clover_description/urdf/sensors/distance_sensor.urdf.xacro (robot description, xacro)
@@ -17,10 +17,12 @@
         </geometry>
       </visual>
+      <!-- remove collision parameters in order to allow for a more realistic minimum range
       <collision>
         <origin xyz="0 0 0" rpy="0 0 0"/>
         <geometry>
-          <box size="0.0015 0.025 0.0175"/> <!-- dimension of Adafruit VL53L4CX -->
+          <box size="0.0015 0.025 0.0175"/>
         </geometry>
       </collision>
+      -->
       <inertial>
         <mass value="0.001"/>
