Commit message: feat: changing description files to match VL53L4CX and leaving fixmes for later

File: clover_description/urdf/clover/clover4.xacro (robot description, xacro)
@@ -3,5 +3,5 @@
   <xacro:arg name="main_camera" default="true"/>
   <xacro:arg name="rangefinder" default="true"/>
-  <xacro:arg name="led" default="true"/>
+  <xacro:arg name="led" default="false"/>
   <xacro:arg name="gps" default="true"/>
   <xacro:arg name="maintain_camera_rate" default="false"/>
@@ -17,5 +17,14 @@
   <!-- Create rangefinder plugin -->
   <xacro:if value="$(arg rangefinder)">
-    <xacro:distance_sensor parent="base_link" x="0.0" y="0.0" z="-0.04" roll="0" pitch="${pi / 2}" yaw="0"/>
+    <xacro:distance_sensor index="0" parent="base_link" x="0.0" y="0.0" z="-0.04" roll="0" pitch="${pi / 2}" yaw="0" range_min="0.001" range_max="6.0"/>
+    <xacro:distance_sensor index="1" parent="base_link" x="0.0" y="0.0" z="-0.04" roll="0" pitch="${pi / 2}" yaw="0" range_min="0.001" range_max="6.0"/>
+    <xacro:distance_sensor index="2" parent="base_link" x="0.0" y="0.0" z="-0.04" roll="0" pitch="${pi / 2}" yaw="0" range_min="0.001" range_max="6.0"/>
+    <xacro:distance_sensor index="3" parent="base_link" x="0.0" y="0.0" z="-0.04" roll="0" pitch="${pi / 2}" yaw="0" range_min="0.001" range_max="6.0"/>
+    <xacro:distance_sensor index="4" parent="base_link" x="0.0" y="0.0" z="-0.04" roll="0" pitch="${pi / 2}" yaw="0" range_min="0.001" range_max="6.0"/>
+    <xacro:distance_sensor index="5" parent="base_link" x="0.0" y="0.0" z="-0.04" roll="0" pitch="${pi / 2}" yaw="0" range_min="0.001" range_max="6.0"/>
+    <xacro:distance_sensor index="6" parent="base_link" x="0.0" y="0.0" z="-0.04" roll="0" pitch="${pi / 2}" yaw="0" range_min="0.001" range_max="6.0"/>
+    <xacro:distance_sensor index="7" parent="base_link" x="0.0" y="0.0" z="-0.04" roll="0" pitch="${pi / 2}" yaw="0" range_min="0.001" range_max="6.0"/>
+    <xacro:distance_sensor index="8" parent="base_link" x="0.0" y="0.0" z="-0.04" roll="0" pitch="${pi / 2}" yaw="0" range_min="0.001" range_max="6.0"/>
+    <xacro:distance_sensor index="9" parent="base_link" x="0.0" y="0.0" z="-0.04" roll="0" pitch="${pi / 2}" yaw="0" range_min="0.001" range_max="6.0"/>
   </xacro:if>
   <!-- Instantiate LED strip -->

File: clover_description/urdf/sensors/distance_sensor.urdf.xacro (robot description, xacro)
@@ -1,6 +1,8 @@
 <?xml version="1.0" encoding="UTF-8"?>
 <robot name="rpi_camera" xmlns:xacro="http://ros.org/wiki/xacro">
+  <xacro:arg name="" default="true"/>
+  <xacro:arg name="" default="true"/>
   <xacro:include filename="../camera_sensor.urdf.xacro"/>
-  <xacro:macro name="distance_sensor" params="name:=lidar_vl53l1x parent x:=0 y:=0 z:=0 roll:=0 pitch:=0 yaw:=0 range_min:=0.01 range_max:=4.0 resolution:=0.01 rate:=10 fov:=0.471239">
+  <xacro:macro name="distance_sensor" params="name:=lidar_VL53L4CX index parent x:=0 y:=0 z:=0 roll:=0 pitch:=0 yaw:=0 range_min range_max resolution:=0.01 rate:=10 fov:=0.3141593">
     <joint name="${name}_joint" type="fixed">
       <origin xyz="${x} ${y} ${z}"
@@ -52,6 +54,6 @@
         <plugin name="laser" filename="libgazebo_ros_range.so">
           <robotNamespace></robotNamespace> <!-- FIXME: fill namespace? -->
-          <topicName>/rangefinder/range</topicName>
-          <frameName>rangefinder</frameName>
+          <topicName>/rangefinder_${index}/range</topicName> <!-- put index here to uniquely identify topics -->
+          <frameName>rangefinder_${index}</frameName>
           <radiation>infrared</radiation>
           <fov>${fov}</fov>

Commit message: feat: distance sensor poses programmatically

File: clover_description/urdf/clover/clover4.xacro (robot description, xacro)
@@ -17,14 +17,22 @@
   <!-- Create rangefinder plugin -->
   <xacro:if value="$(arg rangefinder)">
-    <xacro:distance_sensor index="0" parent="base_link" x="0.0" y="0.0" z="-0.04" roll="0" pitch="${pi / 2}" yaw="0" range_min="0.001" range_max="6.0"/>
-    <xacro:distance_sensor index="1" parent="base_link" x="0.0" y="0.0" z="-0.04" roll="0" pitch="${pi / 2}" yaw="0" range_min="0.001" range_max="6.0"/>
-    <xacro:distance_sensor index="2" parent="base_link" x="0.0" y="0.0" z="-0.04" roll="0" pitch="${pi / 2}" yaw="0" range_min="0.001" range_max="6.0"/>
-    <xacro:distance_sensor index="3" parent="base_link" x="0.0" y="0.0" z="-0.04" roll="0" pitch="${pi / 2}" yaw="0" range_min="0.001" range_max="6.0"/>
-    <xacro:distance_sensor index="4" parent="base_link" x="0.0" y="0.0" z="-0.04" roll="0" pitch="${pi / 2}" yaw="0" range_min="0.001" range_max="6.0"/>
-    <xacro:distance_sensor index="5" parent="base_link" x="0.0" y="0.0" z="-0.04" roll="0" pitch="${pi / 2}" yaw="0" range_min="0.001" range_max="6.0"/>
-    <xacro:distance_sensor index="6" parent="base_link" x="0.0" y="0.0" z="-0.04" roll="0" pitch="${pi / 2}" yaw="0" range_min="0.001" range_max="6.0"/>
-    <xacro:distance_sensor index="7" parent="base_link" x="0.0" y="0.0" z="-0.04" roll="0" pitch="${pi / 2}" yaw="0" range_min="0.001" range_max="6.0"/>
-    <xacro:distance_sensor index="8" parent="base_link" x="0.0" y="0.0" z="-0.04" roll="0" pitch="${pi / 2}" yaw="0" range_min="0.001" range_max="6.0"/>
-    <xacro:distance_sensor index="9" parent="base_link" x="0.0" y="0.0" z="-0.04" roll="0" pitch="${pi / 2}" yaw="0" range_min="0.001" range_max="6.0"/>
+    <!--
+      Radius of tof_sensor_array_drum is 20cm from the center of it.
+      I increment through values of 2pi/8 (8-sided) for the x y positioning of each sensor.
+      Phi is the angular offset, because the faces of the octagon are offset at a 22.5deg angle.
+    -->
+    <xacro:property name="rangefinder_" value="0.2" />
+    <xacro:property name="d_theta" value="${2 * pi / 8}" />
+    <xacro:property name="phi" value="${22.5 * pi / 180}" />
+    <xacro:distance_sensor index="0" parent="tof_sensor_array_link" x="${r*cos((d_theta * 0) + phi)}" y="${r*sin((d_theta * 0) + phi)}" z="-0.04" roll="0" pitch="${pi / 2}" yaw="(d_theta * 0) + phi" range_min="0.001" range_max="6.0"/>
+    <xacro:distance_sensor index="1" parent="tof_sensor_array_link" x="${r*cos((d_theta * 1) + phi)}" y="${r*sin((d_theta * 1) + phi)}" z="-0.04" roll="0" pitch="${pi / 2}" yaw="(d_theta * 1)" range_min="0.001" range_max="6.0"/>
+    <xacro:distance_sensor index="2" parent="tof_sensor_array_link" x="${r*cos((d_theta * 2) + phi)}" y="${r*sin((d_theta * 2) + phi)}" z="-0.04" roll="0" pitch="${pi / 2}" yaw="(d_theta * 2)" range_min="0.001" range_max="6.0"/>
+    <xacro:distance_sensor index="3" parent="tof_sensor_array_link" x="${r*cos((d_theta * 3) + phi)}" y="${r*sin((d_theta * 3) + phi)}" z="-0.04" roll="0" pitch="${pi / 2}" yaw="(d_theta * 3)" range_min="0.001" range_max="6.0"/>
+    <xacro:distance_sensor index="4" parent="tof_sensor_array_link" x="${r*cos((d_theta * 4) + phi)}" y="${r*sin((d_theta * 4) + phi)}" z="-0.04" roll="0" pitch="${pi / 2}" yaw="(d_theta * 4)" range_min="0.001" range_max="6.0"/>
+    <xacro:distance_sensor index="5" parent="tof_sensor_array_link" x="${r*cos((d_theta * 5) + phi)}" y="${r*sin((d_theta * 5) + phi)}" z="-0.04" roll="0" pitch="${pi / 2}" yaw="(d_theta * 5)" range_min="0.001" range_max="6.0"/>
+    <xacro:distance_sensor index="6" parent="tof_sensor_array_link" x="${r*cos((d_theta * 6) + phi)}" y="${r*sin((d_theta * 6) + phi)}" z="-0.04" roll="0" pitch="${pi / 2}" yaw="(d_theta * 6)" range_min="0.001" range_max="6.0"/>
+    <xacro:distance_sensor index="7" parent="tof_sensor_array_link" x="${r*cos((d_theta * 7) + phi)}" y="${r*sin((d_theta * 7) + phi)}" z="-0.04" roll="0" pitch="${pi / 2}" yaw="(d_theta * 7)" range_min="0.001" range_max="6.0"/>
+    <xacro:distance_sensor index="8" parent="base_link" x="0" y="0" z="0.005" roll="0" pitch="${pi / 2}" yaw="0" range_min="0.001" range_max="6.0"/> <!-- up-facing sensor-->
+    <xacro:distance_sensor index="9" parent="tof_sensor_array_link" x="0" y="0" z="-0.05" roll="0" pitch="${pi / 2}" yaw="0" range_min="0.001" range_max="6.0"/> <!-- down-facing sensor -->
   </xacro:if>
   <!-- Instantiate LED strip -->

File: clover_description/urdf/sensors/distance_sensor.urdf.xacro (robot description, xacro)
@@ -1,7 +1,6 @@
 <?xml version="1.0" encoding="UTF-8"?>
-<robot name="rpi_camera" xmlns:xacro="http://ros.org/wiki/xacro">
+<robot name="rpi_rangefinder" xmlns:xacro="http://ros.org/wiki/xacro">
   <xacro:arg name="" default="true"/>
   <xacro:arg name="" default="true"/>
-  <xacro:include filename="../camera_sensor.urdf.xacro"/>
   <xacro:macro name="distance_sensor" params="name:=lidar_VL53L4CX index parent x:=0 y:=0 z:=0 roll:=0 pitch:=0 yaw:=0 range_min range_max resolution:=0.01 rate:=10 fov:=0.3141593">
     <joint name="${name}_${index}_joint" type="fixed">

Commit message: fix: r variable for radius

File: clover_description/urdf/clover/clover4.xacro (robot description, xacro)
@@ -22,5 +22,5 @@
       Phi is the angular offset, because the faces of the octagon are offset at a 22.5deg angle.
     -->
-    <xacro:property name="rangefinder_" value="0.2" />
+    <xacro:property name="r" value="0.2" />
     <xacro:property name="d_theta" value="${2 * pi / 8}" />
     <xacro:property name="phi" value="${22.5 * pi / 180}" />

Commit message: fix: xacro syntax

File: clover_description/urdf/clover/clover4.xacro (robot description, xacro)
@@ -23,14 +23,14 @@
     -->
     <xacro:property name="r" value="0.2" />
-    <xacro:property name="d_theta" value="${2 * pi / 8}" />
-    <xacro:property name="phi" value="${22.5 * pi / 180}" />
-    <xacro:distance_sensor index="0" parent="tof_sensor_array_link" x="${r*cos((d_theta * 0) + phi)}" y="${r*sin((d_theta * 0) + phi)}" z="-0.04" roll="0" pitch="${pi / 2}" yaw="(d_theta * 0) + phi" range_min="0.001" range_max="6.0"/>
-    <xacro:distance_sensor index="1" parent="tof_sensor_array_link" x="${r*cos((d_theta * 1) + phi)}" y="${r*sin((d_theta * 1) + phi)}" z="-0.04" roll="0" pitch="${pi / 2}" yaw="(d_theta * 1)" range_min="0.001" range_max="6.0"/>
-    <xacro:distance_sensor index="2" parent="tof_sensor_array_link" x="${r*cos((d_theta * 2) + phi)}" y="${r*sin((d_theta * 2) + phi)}" z="-0.04" roll="0" pitch="${pi / 2}" yaw="(d_theta * 2)" range_min="0.001" range_max="6.0"/>
-    <xacro:distance_sensor index="3" parent="tof_sensor_array_link" x="${r*cos((d_theta * 3) + phi)}" y="${r*sin((d_theta * 3) + phi)}" z="-0.04" roll="0" pitch="${pi / 2}" yaw="(d_theta * 3)" range_min="0.001" range_max="6.0"/>
-    <xacro:distance_sensor index="4" parent="tof_sensor_array_link" x="${r*cos((d_theta * 4) + phi)}" y="${r*sin((d_theta * 4) + phi)}" z="-0.04" roll="0" pitch="${pi / 2}" yaw="(d_theta * 4)" range_min="0.001" range_max="6.0"/>
-    <xacro:distance_sensor index="5" parent="tof_sensor_array_link" x="${r*cos((d_theta * 5) + phi)}" y="${r*sin((d_theta * 5) + phi)}" z="-0.04" roll="0" pitch="${pi / 2}" yaw="(d_theta * 5)" range_min="0.001" range_max="6.0"/>
-    <xacro:distance_sensor index="6" parent="tof_sensor_array_link" x="${r*cos((d_theta * 6) + phi)}" y="${r*sin((d_theta * 6) + phi)}" z="-0.04" roll="0" pitch="${pi / 2}" yaw="(d_theta * 6)" range_min="0.001" range_max="6.0"/>
-    <xacro:distance_sensor index="7" parent="tof_sensor_array_link" x="${r*cos((d_theta * 7) + phi)}" y="${r*sin((d_theta * 7) + phi)}" z="-0.04" roll="0" pitch="${pi / 2}" yaw="(d_theta * 7)" range_min="0.001" range_max="6.0"/>
+    <xacro:property name="d_theta" value="${2.0 * pi / 8.0}" />
+    <xacro:property name="phi" value="${22.5 * pi / 180.0}" />
+    <xacro:distance_sensor index="0" parent="tof_sensor_array_link" x="${r*cos((d_theta * 0) + phi)}" y="${r*sin((d_theta * 0) + phi)}" z="-0.04" roll="0" pitch="${pi / 2}" yaw="${d_theta * 0 + phi}" range_min="0.001" range_max="6.0"/>
+    <xacro:distance_sensor index="1" parent="tof_sensor_array_link" x="${r*cos((d_theta * 1) + phi)}" y="${r*sin((d_theta * 1) + phi)}" z="-0.04" roll="0" pitch="${pi / 2}" yaw="${d_theta * 1}" range_min="0.001" range_max="6.0"/>
+    <xacro:distance_sensor index="2" parent="tof_sensor_array_link" x="${r*cos((d_theta * 2) + phi)}" y="${r*sin((d_theta * 2) + phi)}" z="-0.04" roll="0" pitch="${pi / 2}" yaw="${d_theta * 2}" range_min="0.001" range_max="6.0"/>
+    <xacro:distance_sensor index="3" parent="tof_sensor_array_link" x="${r*cos((d_theta * 3) + phi)}" y="${r*sin((d_theta * 3) + phi)}" z="-0.04" roll="0" pitch="${pi / 2}" yaw="${d_theta * 3}" range_min="0.001" range_max="6.0"/>
+    <xacro:distance_sensor index="4" parent="tof_sensor_array_link" x="${r*cos((d_theta * 4) + phi)}" y="${r*sin((d_theta * 4) + phi)}" z="-0.04" roll="0" pitch="${pi / 2}" yaw="${d_theta * 4}" range_min="0.001" range_max="6.0"/>
+    <xacro:distance_sensor index="5" parent="tof_sensor_array_link" x="${r*cos((d_theta * 5) + phi)}" y="${r*sin((d_theta * 5) + phi)}" z="-0.04" roll="0" pitch="${pi / 2}" yaw="${d_theta * 5}" range_min="0.001" range_max="6.0"/>
+    <xacro:distance_sensor index="6" parent="tof_sensor_array_link" x="${r*cos((d_theta * 6) + phi)}" y="${r*sin((d_theta * 6) + phi)}" z="-0.04" roll="0" pitch="${pi / 2}" yaw="${d_theta * 6}" range_min="0.001" range_max="6.0"/>
+    <xacro:distance_sensor index="7" parent="tof_sensor_array_link" x="${r*cos((d_theta * 7) + phi)}" y="${r*sin((d_theta * 7) + phi)}" z="-0.04" roll="0" pitch="${pi / 2}" yaw="${d_theta * 7}" range_min="0.001" range_max="6.0"/>
     <xacro:distance_sensor index="8" parent="base_link" x="0" y="0" z="0.005" roll="0" pitch="${pi / 2}" yaw="0" range_min="0.001" range_max="6.0"/> <!-- up-facing sensor-->
     <xacro:distance_sensor index="9" parent="tof_sensor_array_link" x="0" y="0" z="-0.05" roll="0" pitch="${pi / 2}" yaw="0" range_min="0.001" range_max="6.0"/> <!-- down-facing sensor -->

Commit message: fix: radius of tof drum

File: clover_description/urdf/clover/clover4.xacro (robot description, xacro)
@@ -22,5 +22,5 @@
       Phi is the angular offset, because the faces of the octagon are offset at a 22.5deg angle.
     -->
-    <xacro:property name="r" value="0.2" />
+    <xacro:property name="r" value="0.05" />
     <xacro:property name="d_theta" value="${2.0 * pi / 8.0}" />
     <xacro:property name="phi" value="${22.5 * pi / 180.0}" />

Commit message: feat: gazebo minimum range tweaking

File: clover_description/urdf/clover/clover4.xacro (robot description, xacro)
@@ -33,6 +33,6 @@
     <xacro:distance_sensor index="6" parent="tof_sensor_array_link" x="${r*cos((d_theta * 6) + phi)}" y="${r*sin((d_theta * 6) + phi)}" z="-0.04" roll="0" pitch="${0}" yaw="${d_theta * 6 + phi}" range_min="0.001" range_max="6.0"/>
     <xacro:distance_sensor index="7" parent="tof_sensor_array_link" x="${r*cos((d_theta * 7) + phi)}" y="${r*sin((d_theta * 7) + phi)}" z="-0.04" roll="0" pitch="${0}" yaw="${d_theta * 7 + phi}" range_min="0.001" range_max="6.0"/>
-    <xacro:distance_sensor index="8" parent="base_link" x="0" y="0" z="0.005" roll="0" pitch="${pi / 2}" yaw="0" range_min="0.001" range_max="6.0"/> <!-- up-facing sensor-->
-    <xacro:distance_sensor index="9" parent="tof_sensor_array_link" x="0" y="0" z="-0.05" roll="0" pitch="${3 * pi / 2}" yaw="0" range_min="0.001" range_max="6.0"/> <!-- down-facing sensor -->
+    <xacro:distance_sensor index="8" parent="base_link" x="0" y="0" z="0.05" roll="0" pitch="${pi / 2}" yaw="0" range_min="0.001" range_min_gazebo="0.01" range_max="6.0"/> <!-- up-facing sensor-->
+    <xacro:distance_sensor index="9" parent="tof_sensor_array_link" x="0" y="0" z="-0.05" roll="0" pitch="${3 * pi / 2}" yaw="0" range_min="0.001" range_min_gazebo="0.01" range_max="6.0"/> <!-- down-facing sensor -->
   </xacro:if>
   <!-- Instantiate LED strip -->

File: clover_description/urdf/sensors/distance_sensor.urdf.xacro (robot description, xacro)
@@ -3,5 +3,5 @@
   <xacro:arg name="" default="true"/>
   <xacro:arg name="" default="true"/>
-  <xacro:macro name="distance_sensor" params="name:=lidar_VL53L4CX index parent x:=0 y:=0 z:=0 roll:=0 pitch:=0 yaw:=0 range_min range_max resolution:=0.01 rate:=10 fov:=0.3141593">
+  <xacro:macro name="distance_sensor" params="name:=lidar_VL53L4CX index parent x:=0 y:=0 z:=0 roll:=0 pitch:=0 yaw:=0 range_min range_min_gazebo:=0.2 range_max resolution:=0.01 rate:=10 fov:=0.3141593">
     <joint name="${name}_${index}_joint" type="fixed">
       <origin xyz="${x} ${y} ${z}"
@@ -46,5 +46,5 @@
           </scan>
           <range>
-            <min>0.2</min> <!-- Note: This is a hack, since the rangefinder is inside the drone collision box -->
+            <min>${range_min_gazebo}</min> <!-- Note: This is a hack, since the rangefinder is inside the drone collision box -->
             <max>${range_max}</max>
             <resolution>${resolution}</resolution>

Commit message: feat: tof_sensor_drum positioning

File: clover_description/urdf/clover/clover4.xacro (robot description, xacro)
@@ -33,5 +33,5 @@
     <xacro:distance_sensor index="6" parent="tof_sensor_array_link" x="${r*cos((d_theta * 6) + phi)}" y="${r*sin((d_theta * 6) + phi)}" z="-0.04" roll="0" pitch="${0}" yaw="${d_theta * 6 + phi}" range_min="0.001" range_max="6.0"/>
     <xacro:distance_sensor index="7" parent="tof_sensor_array_link" x="${r*cos((d_theta * 7) + phi)}" y="${r*sin((d_theta * 7) + phi)}" z="-0.04" roll="0" pitch="${0}" yaw="${d_theta * 7 + phi}" range_min="0.001" range_max="6.0"/>
-    <xacro:distance_sensor index="8" parent="base_link" x="0" y="0" z="0.05" roll="0" pitch="${pi / 2}" yaw="0" range_min="0.001" range_min_gazebo="0.015" range_max="6.0"/> <!-- up-facing sensor-->
+    <xacro:distance_sensor index="8" parent="base_link" x="0" y="0" z="0.075" roll="0" pitch="${pi / 2}" yaw="0" range_min="0.001" range_min_gazebo="0.015" range_max="6.0"/> <!-- up-facing sensor-->
     <xacro:distance_sensor index="9" parent="tof_sensor_array_link" x="0" y="0" z="-0.05" roll="0" pitch="${3 * pi / 2}" yaw="0" range_min="0.001" range_min_gazebo="0.015" range_max="6.0"/> <!-- down-facing sensor -->
   </xacro:if>

File: clover_description/urdf/clover/clover4_macros.xacro (robot description, xacro)
@@ -128,5 +128,5 @@
       <inertial>
         <mass value="0.092"/> <!-- [kg] -->
-        <origin xyz="0 0 ${-1 * 0.01525 / 2}" rpy="0 0 0"/>
+        <origin xyz="0 0 -0.015" rpy="0 0 0"/>
         <inertia
           ixx="8.57890084602841e-5"

Commit message: feat: custom translation in the x direction for rpi camera to avoid sensor drum

File: clover_description/urdf/clover/clover4.xacro (robot description, xacro)
@@ -13,5 +13,6 @@
   <!-- Create camera plugin -->
   <xacro:if value="$(arg main_camera)">
-    <xacro:rpi_cam name="main_camera" parent="base_link" x="0.055" y="0.0" z="-0.03" roll="0" pitch="${pi / 2}" yaw="0" width="320" height="240" rate="40" do_throttling="$(arg maintain_camera_rate)"/>
+    <xacro:property name="rpi_cam_x_translation" value="0.02" /> <!-- custom translation of rpi cam to make it -->
+    <xacro:rpi_cam name="main_camera" parent="base_link" x="${0.055 + rpi_cam_x_translation}" y="0.0" z="-0.03" roll="0" pitch="${pi / 2}" yaw="0" width="320" height="240" rate="40" do_throttling="$(arg maintain_camera_rate)"/>
   </xacro:if>
   <!-- Create rangefinder plugin -->

Commit message: feat: adjusting rpi camera x translation larger

File: clover_description/urdf/clover/clover4.xacro (robot description, xacro)
@@ -13,5 +13,5 @@
   <!-- Create camera plugin -->
   <xacro:if value="$(arg main_camera)">
-    <xacro:property name="rpi_cam_x_translation" value="0.02" /> <!-- custom translation of rpi cam to make it -->
+    <xacro:property name="rpi_cam_x_translation" value="0.04" /> <!-- custom translation of rpi cam to make it -->
     <xacro:rpi_cam name="main_camera" parent="base_link" x="${0.055 + rpi_cam_x_translation}" y="0.0" z="-0.03" roll="0" pitch="${pi / 2}" yaw="0" width="320" height="240" rate="40" do_throttling="$(arg maintain_camera_rate)"/>
   </xacro:if>
