Commit message: feat: tof sensor array position

File: clover_description/urdf/clover/clover4.xacro (robot description, xacro)
@@ -26,12 +26,12 @@
     <xacro:property name="d_theta" value="${2.0 * pi / 8.0}" />
     <xacro:property name="phi" value="${22.5 * pi / 180.0}" />
-    <xacro:distance_sensor index="0" parent="tof_sensor_array_link" x="${r*cos((d_theta * 0) + phi)}" y="${r*sin((d_theta * 0) + phi)}" z="-0.04" roll="0" pitch="${0}" yaw="${d_theta * 0 + phi}" range_min="0.001" range_max="6.0"/>
-    <xacro:distance_sensor index="1" parent="tof_sensor_array_link" x="${r*cos((d_theta * 1) + phi)}" y="${r*sin((d_theta * 1) + phi)}" z="-0.04" roll="0" pitch="${0}" yaw="${d_theta * 1 + phi}" range_min="0.001" range_max="6.0"/>
-    <xacro:distance_sensor index="2" parent="tof_sensor_array_link" x="${r*cos((d_theta * 2) + phi)}" y="${r*sin((d_theta * 2) + phi)}" z="-0.04" roll="0" pitch="${0}" yaw="${d_theta * 2 + phi}" range_min="0.001" range_max="6.0"/>
-    <xacro:distance_sensor index="3" parent="tof_sensor_array_link" x="${r*cos((d_theta * 3) + phi)}" y="${r*sin((d_theta * 3) + phi)}" z="-0.04" roll="0" pitch="${0}" yaw="${d_theta * 3 + phi}" range_min="0.001" range_max="6.0"/>
-    <xacro:distance_sensor index="4" parent="tof_sensor_array_link" x="${r*cos((d_theta * 4) + phi)}" y="${r*sin((d_theta * 4) + phi)}" z="-0.04" roll="0" pitch="${0}" yaw="${d_theta * 4 + phi}" range_min="0.001" range_max="6.0"/>
-    <xacro:distance_sensor index="5" parent="tof_sensor_array_link" x="${r*cos((d_theta * 5) + phi)}" y="${r*sin((d_theta * 5) + phi)}" z="-0.04" roll="0" pitch="${0}" yaw="${d_theta * 5 + phi}" range_min="0.001" range_max="6.0"/>
-    <xacro:distance_sensor index="6" parent="tof_sensor_array_link" x="${r*cos((d_theta * 6) + phi)}" y="${r*sin((d_theta * 6) + phi)}" z="-0.04" roll="0" pitch="${0}" yaw="${d_theta * 6 + phi}" range_min="0.001" range_max="6.0"/>
-    <xacro:distance_sensor index="7" parent="tof_sensor_array_link" x="${r*cos((d_theta * 7) + phi)}" y="${r*sin((d_theta * 7) + phi)}" z="-0.04" roll="0" pitch="${0}" yaw="${d_theta * 7 + phi}" range_min="0.001" range_max="6.0"/>
+    <xacro:distance_sensor index="0" parent="tof_sensor_array_link" x="${r*cos((d_theta * 0) + phi)}" y="${r*sin((d_theta * 0) + phi)}" z="0" roll="0" pitch="${0}" yaw="${d_theta * 0 + phi}" range_min="0.001" range_max="6.0"/>
+    <xacro:distance_sensor index="1" parent="tof_sensor_array_link" x="${r*cos((d_theta * 1) + phi)}" y="${r*sin((d_theta * 1) + phi)}" z="0" roll="0" pitch="${0}" yaw="${d_theta * 1 + phi}" range_min="0.001" range_max="6.0"/>
+    <xacro:distance_sensor index="2" parent="tof_sensor_array_link" x="${r*cos((d_theta * 2) + phi)}" y="${r*sin((d_theta * 2) + phi)}" z="0" roll="0" pitch="${0}" yaw="${d_theta * 2 + phi}" range_min="0.001" range_max="6.0"/>
+    <xacro:distance_sensor index="3" parent="tof_sensor_array_link" x="${r*cos((d_theta * 3) + phi)}" y="${r*sin((d_theta * 3) + phi)}" z="0" roll="0" pitch="${0}" yaw="${d_theta * 3 + phi}" range_min="0.001" range_max="6.0"/>
+    <xacro:distance_sensor index="4" parent="tof_sensor_array_link" x="${r*cos((d_theta * 4) + phi)}" y="${r*sin((d_theta * 4) + phi)}" z="0" roll="0" pitch="${0}" yaw="${d_theta * 4 + phi}" range_min="0.001" range_max="6.0"/>
+    <xacro:distance_sensor index="5" parent="tof_sensor_array_link" x="${r*cos((d_theta * 5) + phi)}" y="${r*sin((d_theta * 5) + phi)}" z="0" roll="0" pitch="${0}" yaw="${d_theta * 5 + phi}" range_min="0.001" range_max="6.0"/>
+    <xacro:distance_sensor index="6" parent="tof_sensor_array_link" x="${r*cos((d_theta * 6) + phi)}" y="${r*sin((d_theta * 6) + phi)}" z="0" roll="0" pitch="${0}" yaw="${d_theta * 6 + phi}" range_min="0.001" range_max="6.0"/>
+    <xacro:distance_sensor index="7" parent="tof_sensor_array_link" x="${r*cos((d_theta * 7) + phi)}" y="${r*sin((d_theta * 7) + phi)}" z="0" roll="0" pitch="${0}" yaw="${d_theta * 7 + phi}" range_min="0.001" range_max="6.0"/>
     <xacro:distance_sensor index="8" parent="base_link" x="0" y="0" z="0.1" roll="0" pitch="${3 * pi / 2}" yaw="0" range_min="0.001" range_min_gazebo="0.015" range_max="6.0"/> <!-- up-facing sensor-->
     <xacro:distance_sensor index="9" parent="tof_sensor_array_link" x="0" y="0" z="-0.05" roll="0" pitch="${pi / 2}" yaw="0" range_min="0.001" range_min_gazebo="0.02" range_max="6.0"/> <!-- down-facing sensor -->

File: clover_description/urdf/clover/clover4_macros.xacro (robot description, xacro)
@@ -124,9 +124,8 @@
     </joint>
     <!-- FIXME: how to set origin correctly? -->
-    <!-- FIXME: how to add rangefinder sensors? -->
     <link name="tof_sensor_array_link">
       <inertial>
         <mass value="0.092"/> <!-- [kg] -->
-        <origin xyz="0 0 -0.015" rpy="0 0 0"/>
+        <origin xyz="0 0 0" rpy="0 0 0"/>
         <inertia
           ixx="8.57890084602841e-5"
@@ -139,5 +138,5 @@
       </inertial>
       <collision>
-        <origin xyz="0 0 -0.015" rpy="0 0 0" />
+        <origin xyz="0 0 0" rpy="0 0 0" />
         <geometry>
           <box size=".101567337 .101567337 .030500050" /> <!-- [m] [m] [m] -->
@@ -145,13 +144,13 @@
       </collision>
       <visual>
-        <origin xyz="0 0 -0.015" rpy="0 0 0"/>
+        <origin xyz="0 0 0" rpy="0 0 0"/>
         <geometry>
           <mesh filename="package://clover_description/meshes/clover4/tof_sensor_drum.dae"
-            scale="0.01 0.01 0.01"/> <!-- scale down because model is represented in mm -->
+            scale="1 1 1"/> <!-- scale down because model is represented in mm -->
         </geometry>
       </visual>
     </link>
     <joint name="tof_sensor_array_joint" type="fixed">
-      <origin xyz="0 0 -0.015" rpy="0 0 0"/>
+      <origin xyz="0 0 -0.05" rpy="0 0 0"/>
       <parent link="base_link" />
       <child link="tof_sensor_array_link" />

Commit message: feat: tof distance sensors position

File: clover_description/urdf/clover/clover4.xacro (robot description, xacro)
@@ -26,14 +26,14 @@
     <xacro:property name="d_theta" value="${2.0 * pi / 8.0}" />
     <xacro:property name="phi" value="${22.5 * pi / 180.0}" />
-    <xacro:distance_sensor index="0" parent="tof_sensor_array_link" x="${r*cos((d_theta * 0) + phi)}" y="${r*sin((d_theta * 0) + phi)}" z="0" roll="0" pitch="${0}" yaw="${d_theta * 0 + phi}" range_min="0.001" range_max="6.0"/>
-    <xacro:distance_sensor index="1" parent="tof_sensor_array_link" x="${r*cos((d_theta * 1) + phi)}" y="${r*sin((d_theta * 1) + phi)}" z="0" roll="0" pitch="${0}" yaw="${d_theta * 1 + phi}" range_min="0.001" range_max="6.0"/>
-    <xacro:distance_sensor index="2" parent="tof_sensor_array_link" x="${r*cos((d_theta * 2) + phi)}" y="${r*sin((d_theta * 2) + phi)}" z="0" roll="0" pitch="${0}" yaw="${d_theta * 2 + phi}" range_min="0.001" range_max="6.0"/>
-    <xacro:distance_sensor index="3" parent="tof_sensor_array_link" x="${r*cos((d_theta * 3) + phi)}" y="${r*sin((d_theta * 3) + phi)}" z="0" roll="0" pitch="${0}" yaw="${d_theta * 3 + phi}" range_min="0.001" range_max="6.0"/>
-    <xacro:distance_sensor index="4" parent="tof_sensor_array_link" x="${r*cos((d_theta * 4) + phi)}" y="${r*sin((d_theta * 4) + phi)}" z="0" roll="0" pitch="${0}" yaw="${d_theta * 4 + phi}" range_min="0.001" range_max="6.0"/>
-    <xacro:distance_sensor index="5" parent="tof_sensor_array_link" x="${r*cos((d_theta * 5) + phi)}" y="${r*sin((d_theta * 5) + phi)}" z="0" roll="0" pitch="${0}" yaw="${d_theta * 5 + phi}" range_min="0.001" range_max="6.0"/>
-    <xacro:distance_sensor index="6" parent="tof_sensor_array_link" x="${r*cos((d_theta * 6) + phi)}" y="${r*sin((d_theta * 6) + phi)}" z="0" roll="0" pitch="${0}" yaw="${d_theta * 6 + phi}" range_min="0.001" range_max="6.0"/>
-    <xacro:distance_sensor index="7" parent="tof_sensor_array_link" x="${r*cos((d_theta * 7) + phi)}" y="${r*sin((d_theta * 7) + phi)}" z="0" roll="0" pitch="${0}" yaw="${d_theta * 7 + phi}" range_min="0.001" range_max="6.0"/>
+    <xacro:distance_sensor index="0" parent="tof_sensor_array_link" x="${r*cos((d_theta * 0) + phi)}" y="${r*sin((d_theta * 0) + phi)}" z="${-0.0175 / 2}" roll="0" pitch="${0}" yaw="${d_theta * 0 + phi}" range_min="0.001" range_max="6.0"/>
+    <xacro:distance_sensor index="1" parent="tof_sensor_array_link" x="${r*cos((d_theta * 1) + phi)}" y="${r*sin((d_theta * 1) + phi)}" z="${-0.0175 / 2}" roll="0" pitch="${0}" yaw="${d_theta * 1 + phi}" range_min="0.001" range_max="6.0"/>
+    <xacro:distance_sensor index="2" parent="tof_sensor_array_link" x="${r*cos((d_theta * 2) + phi)}" y="${r*sin((d_theta * 2) + phi)}" z="${-0.0175 / 2}" roll="0" pitch="${0}" yaw="${d_theta * 2 + phi}" range_min="0.001" range_max="6.0"/>
+    <xacro:distance_sensor index="3" parent="tof_sensor_array_link" x="${r*cos((d_theta * 3) + phi)}" y="${r*sin((d_theta * 3) + phi)}" z="${-0.0175 / 2}" roll="0" pitch="${0}" yaw="${d_theta * 3 + phi}" range_min="0.001" range_max="6.0"/>
+    <xacro:distance_sensor index="4" parent="tof_sensor_array_link" x="${r*cos((d_theta * 4) + phi)}" y="${r*sin((d_theta * 4) + phi)}" z="${-0.0175 / 2}" roll="0" pitch="${0}" yaw="${d_theta * 4 + phi}" range_min="0.001" range_max="6.0"/>
+    <xacro:distance_sensor index="5" parent="tof_sensor_array_link" x="${r*cos((d_theta * 5) + phi)}" y="${r*sin((d_theta * 5) + phi)}" z="${-0.0175 / 2}" roll="0" pitch="${0}" yaw="${d_theta * 5 + phi}" range_min="0.001" range_max="6.0"/>
+    <xacro:distance_sensor index="6" parent="tof_sensor_array_link" x="${r*cos((d_theta * 6) + phi)}" y="${r*sin((d_theta * 6) + phi)}" z="${-0.0175 / 2}" roll="0" pitch="${0}" yaw="${d_theta * 6 + phi}" range_min="0.001" range_max="6.0"/>
+    <xacro:distance_sensor index="7" parent="tof_sensor_array_link" x="${r*cos((d_theta * 7) + phi)}" y="${r*sin((d_theta * 7) + phi)}" z="${-0.0175 / 2}" roll="0" pitch="${0}" yaw="${d_theta * 7 + phi}" range_min="0.001" range_max="6.0"/>
     <xacro:distance_sensor index="8" parent="base_link" x="0" y="0" z="0.1" roll="0" pitch="${3 * pi / 2}" yaw="0" range_min="0.001" range_min_gazebo="0.015" range_max="6.0"/> <!-- up-facing sensor-->
-    <xacro:distance_sensor index="9" parent="tof_sensor_array_link" x="0" y="0" z="-0.05" roll="0" pitch="${pi / 2}" yaw="0" range_min="0.001" range_min_gazebo="0.02" range_max="6.0"/> <!-- down-facing sensor -->
+    <xacro:distance_sensor index="9" parent="tof_sensor_array_link" x="0" y="0" z="-0.01" roll="0" pitch="${pi / 2}" yaw="0" range_min="0.001" range_min_gazebo="0.02" range_max="6.0"/> <!-- down-facing sensor -->
   </xacro:if>
   <!-- Instantiate LED strip -->

File: clover_description/urdf/sensors/distance_sensor.urdf.xacro (robot description, xacro)
@@ -36,4 +36,5 @@
     </gazebo>
     <gazebo reference="${name}_${index}_link">
+      <material>flatblack</material> <!-- custom material. can be found in clover_description/media/materials/scripts/flatblack.material -->
       <sensor type="ray" name="${name}_${index}">
         <pose>0 0 0 0 0 0</pose>

Commit message: feat: sensor heads aligning wip

File: clover_description/urdf/clover/clover4.xacro (robot description, xacro)
@@ -26,14 +26,14 @@
     <xacro:property name="d_theta" value="${2.0 * pi / 8.0}" />
     <xacro:property name="phi" value="${22.5 * pi / 180.0}" />
-    <xacro:distance_sensor index="0" parent="tof_sensor_array_link" x="${r*cos((d_theta * 0) + phi)}" y="${r*sin((d_theta * 0) + phi)}" z="${-0.0175 / 2}" roll="0" pitch="${0}" yaw="${d_theta * 0 + phi}" range_min="0.001" range_max="6.0"/>
-    <xacro:distance_sensor index="1" parent="tof_sensor_array_link" x="${r*cos((d_theta * 1) + phi)}" y="${r*sin((d_theta * 1) + phi)}" z="${-0.0175 / 2}" roll="0" pitch="${0}" yaw="${d_theta * 1 + phi}" range_min="0.001" range_max="6.0"/>
-    <xacro:distance_sensor index="2" parent="tof_sensor_array_link" x="${r*cos((d_theta * 2) + phi)}" y="${r*sin((d_theta * 2) + phi)}" z="${-0.0175 / 2}" roll="0" pitch="${0}" yaw="${d_theta * 2 + phi}" range_min="0.001" range_max="6.0"/>
-    <xacro:distance_sensor index="3" parent="tof_sensor_array_link" x="${r*cos((d_theta * 3) + phi)}" y="${r*sin((d_theta * 3) + phi)}" z="${-0.0175 / 2}" roll="0" pitch="${0}" yaw="${d_theta * 3 + phi}" range_min="0.001" range_max="6.0"/>
-    <xacro:distance_sensor index="4" parent="tof_sensor_array_link" x="${r*cos((d_theta * 4) + phi)}" y="${r*sin((d_theta * 4) + phi)}" z="${-0.0175 / 2}" roll="0" pitch="${0}" yaw="${d_theta * 4 + phi}" range_min="0.001" range_max="6.0"/>
-    <xacro:distance_sensor index="5" parent="tof_sensor_array_link" x="${r*cos((d_theta * 5) + phi)}" y="${r*sin((d_theta * 5) + phi)}" z="${-0.0175 / 2}" roll="0" pitch="${0}" yaw="${d_theta * 5 + phi}" range_min="0.001" range_max="6.0"/>
-    <xacro:distance_sensor index="6" parent="tof_sensor_array_link" x="${r*cos((d_theta * 6) + phi)}" y="${r*sin((d_theta * 6) + phi)}" z="${-0.0175 / 2}" roll="0" pitch="${0}" yaw="${d_theta * 6 + phi}" range_min="0.001" range_max="6.0"/>
-    <xacro:distance_sensor index="7" parent="tof_sensor_array_link" x="${r*cos((d_theta * 7) + phi)}" y="${r*sin((d_theta * 7) + phi)}" z="${-0.0175 / 2}" roll="0" pitch="${0}" yaw="${d_theta * 7 + phi}" range_min="0.001" range_max="6.0"/>
+    <xacro:distance_sensor index="0" parent="tof_sensor_array_link" x="${r*cos((d_theta * 0) + phi)}" y="${r*sin((d_theta * 0) + phi)}" z="${-0.0175 / 2 + 0.025}" roll="0" pitch="${0}" yaw="${d_theta * 0 + phi}" range_min="0.001" range_max="6.0"/>
+    <xacro:distance_sensor index="1" parent="tof_sensor_array_link" x="${r*cos((d_theta * 1) + phi)}" y="${r*sin((d_theta * 1) + phi)}" z="${-0.0175 / 2 + 0.025}" roll="0" pitch="${0}" yaw="${d_theta * 1 + phi}" range_min="0.001" range_max="6.0"/>
+    <xacro:distance_sensor index="2" parent="tof_sensor_array_link" x="${r*cos((d_theta * 2) + phi)}" y="${r*sin((d_theta * 2) + phi)}" z="${-0.0175 / 2 + 0.025}" roll="0" pitch="${0}" yaw="${d_theta * 2 + phi}" range_min="0.001" range_max="6.0"/>
+    <xacro:distance_sensor index="3" parent="tof_sensor_array_link" x="${r*cos((d_theta * 3) + phi)}" y="${r*sin((d_theta * 3) + phi)}" z="${-0.0175 / 2 + 0.025}" roll="0" pitch="${0}" yaw="${d_theta * 3 + phi}" range_min="0.001" range_max="6.0"/>
+    <xacro:distance_sensor index="4" parent="tof_sensor_array_link" x="${r*cos((d_theta * 4) + phi)}" y="${r*sin((d_theta * 4) + phi)}" z="${-0.0175 / 2 + 0.025}" roll="0" pitch="${0}" yaw="${d_theta * 4 + phi}" range_min="0.001" range_max="6.0"/>
+    <xacro:distance_sensor index="5" parent="tof_sensor_array_link" x="${r*cos((d_theta * 5) + phi)}" y="${r*sin((d_theta * 5) + phi)}" z="${-0.0175 / 2 + 0.025}" roll="0" pitch="${0}" yaw="${d_theta * 5 + phi}" range_min="0.001" range_max="6.0"/>
+    <xacro:distance_sensor index="6" parent="tof_sensor_array_link" x="${r*cos((d_theta * 6) + phi)}" y="${r*sin((d_theta * 6) + phi)}" z="${-0.0175 / 2 + 0.025}" roll="0" pitch="${0}" yaw="${d_theta * 6 + phi}" range_min="0.001" range_max="6.0"/>
+    <xacro:distance_sensor index="7" parent="tof_sensor_array_link" x="${r*cos((d_theta * 7) + phi)}" y="${r*sin((d_theta * 7) + phi)}" z="${-0.0175 / 2 + 0.025}" roll="0" pitch="${0}" yaw="${d_theta * 7 + phi}" range_min="0.001" range_max="6.0"/>
     <xacro:distance_sensor index="8" parent="base_link" x="0" y="0" z="0.1" roll="0" pitch="${3 * pi / 2}" yaw="0" range_min="0.001" range_min_gazebo="0.015" range_max="6.0"/> <!-- up-facing sensor-->
-    <xacro:distance_sensor index="9" parent="tof_sensor_array_link" x="0" y="0" z="-0.01" roll="0" pitch="${pi / 2}" yaw="0" range_min="0.001" range_min_gazebo="0.02" range_max="6.0"/> <!-- down-facing sensor -->
+    <xacro:distance_sensor index="9" parent="tof_sensor_array_link" x="0" y="0" z="${-0.0175 + 0.025}" roll="0" pitch="${pi / 2}" yaw="0" range_min="0.001" range_min_gazebo="0.02" range_max="6.0"/> <!-- down-facing sensor -->
   </xacro:if>
   <!-- Instantiate LED strip -->

File: clover_description/urdf/clover/clover4_macros.xacro (robot description, xacro)
@@ -152,5 +152,5 @@
     </link>
     <joint name="tof_sensor_array_joint" type="fixed">
-      <origin xyz="0 0 -0.05" rpy="0 0 0"/>
+      <origin xyz="0 0 -0.075" rpy="0 0 0"/>
       <parent link="base_link" />
       <child link="tof_sensor_array_link" />

Commit message: feat: sensor heads aligning wip

File: clover_description/urdf/clover/clover4.xacro (robot description, xacro)
@@ -35,5 +35,5 @@
     <xacro:distance_sensor index="7" parent="tof_sensor_array_link" x="${r*cos((d_theta * 7) + phi)}" y="${r*sin((d_theta * 7) + phi)}" z="${-0.0175 / 2 + 0.025}" roll="0" pitch="${0}" yaw="${d_theta * 7 + phi}" range_min="0.001" range_max="6.0"/>
     <xacro:distance_sensor index="8" parent="base_link" x="0" y="0" z="0.1" roll="0" pitch="${3 * pi / 2}" yaw="0" range_min="0.001" range_min_gazebo="0.015" range_max="6.0"/> <!-- up-facing sensor-->
-    <xacro:distance_sensor index="9" parent="tof_sensor_array_link" x="0" y="0" z="${-0.0175 + 0.025}" roll="0" pitch="${pi / 2}" yaw="0" range_min="0.001" range_min_gazebo="0.02" range_max="6.0"/> <!-- down-facing sensor -->
+    <xacro:distance_sensor index="9" parent="tof_sensor_array_link" x="0" y="0" z="${-0.0175 / 2 + 0.025}" roll="0" pitch="${pi / 2}" yaw="0" range_min="0.001" range_min_gazebo="0.02" range_max="6.0"/> <!-- down-facing sensor -->
   </xacro:if>
   <!-- Instantiate LED strip -->

File: clover_description/urdf/clover/clover4_macros.xacro (robot description, xacro)
@@ -151,6 +151,7 @@
       </visual>
     </link>
+    <xacro:property name="tof_sensor_drum_yaw_translate" value="${pi / 2 - pi / 8}" />
     <joint name="tof_sensor_array_joint" type="fixed">
-      <origin xyz="0 0 -0.075" rpy="0 0 0"/>
+      <origin xyz="0 0 -0.07" rpy="0 0 ${tof_sensor_drum_yaw_translate}"/>
       <parent link="base_link" />
       <child link="tof_sensor_array_link" />

Commit message: feat: sensor heads aligning wip

File: clover_description/urdf/clover/clover4.xacro (robot description, xacro)
@@ -25,5 +25,5 @@
     <xacro:property name="r" value="0.05" />
     <xacro:property name="d_theta" value="${2.0 * pi / 8.0}" />
-    <xacro:property name="phi" value="${22.5 * pi / 180.0}" />
+    <xacro:property name="phi" value="${0}" />
     <xacro:distance_sensor index="0" parent="tof_sensor_array_link" x="${r*cos((d_theta * 0) + phi)}" y="${r*sin((d_theta * 0) + phi)}" z="${-0.0175 / 2 + 0.025}" roll="0" pitch="${0}" yaw="${d_theta * 0 + phi}" range_min="0.001" range_max="6.0"/>
     <xacro:distance_sensor index="1" parent="tof_sensor_array_link" x="${r*cos((d_theta * 1) + phi)}" y="${r*sin((d_theta * 1) + phi)}" z="${-0.0175 / 2 + 0.025}" roll="0" pitch="${0}" yaw="${d_theta * 1 + phi}" range_min="0.001" range_max="6.0"/>
@@ -35,5 +35,5 @@
     <xacro:distance_sensor index="7" parent="tof_sensor_array_link" x="${r*cos((d_theta * 7) + phi)}" y="${r*sin((d_theta * 7) + phi)}" z="${-0.0175 / 2 + 0.025}" roll="0" pitch="${0}" yaw="${d_theta * 7 + phi}" range_min="0.001" range_max="6.0"/>
     <xacro:distance_sensor index="8" parent="base_link" x="0" y="0" z="0.1" roll="0" pitch="${3 * pi / 2}" yaw="0" range_min="0.001" range_min_gazebo="0.015" range_max="6.0"/> <!-- up-facing sensor-->
-    <xacro:distance_sensor index="9" parent="tof_sensor_array_link" x="0" y="0" z="${-0.0175 / 2 + 0.025}" roll="0" pitch="${pi / 2}" yaw="0" range_min="0.001" range_min_gazebo="0.02" range_max="6.0"/> <!-- down-facing sensor -->
+    <xacro:distance_sensor index="9" parent="tof_sensor_array_link" x="0" y="0" z="${0}" roll="0" pitch="${pi / 2}" yaw="0" range_min="0.001" range_min_gazebo="0.02" range_max="6.0"/> <!-- down-facing sensor -->
   </xacro:if>
   <!-- Instantiate LED strip -->
