Commit message: feat: sensor heads aligning wip

File: clover_description/urdf/clover/clover4.xacro (robot description, xacro)
@@ -26,14 +26,14 @@
     <xacro:property name="d_theta" value="${2.0 * pi / 8.0}" />
     <xacro:property name="phi" value="${0}" />
-    <xacro:distance_sensor index="0" parent="tof_sensor_array_link" x="${r*cos((d_theta * 0) + phi)}" y="${r*sin((d_theta * 0) + phi)}" z="${-0.0175 / 2 + 0.025}" roll="0" pitch="${0}" yaw="${d_theta * 0 + phi}" range_min="0.001" range_max="6.0"/>
-    <xacro:distance_sensor index="1" parent="tof_sensor_array_link" x="${r*cos((d_theta * 1) + phi)}" y="${r*sin((d_theta * 1) + phi)}" z="${-0.0175 / 2 + 0.025}" roll="0" pitch="${0}" yaw="${d_theta * 1 + phi}" range_min="0.001" range_max="6.0"/>
-    <xacro:distance_sensor index="2" parent="tof_sensor_array_link" x="${r*cos((d_theta * 2) + phi)}" y="${r*sin((d_theta * 2) + phi)}" z="${-0.0175 / 2 + 0.025}" roll="0" pitch="${0}" yaw="${d_theta * 2 + phi}" range_min="0.001" range_max="6.0"/>
-    <xacro:distance_sensor index="3" parent="tof_sensor_array_link" x="${r*cos((d_theta * 3) + phi)}" y="${r*sin((d_theta * 3) + phi)}" z="${-0.0175 / 2 + 0.025}" roll="0" pitch="${0}" yaw="${d_theta * 3 + phi}" range_min="0.001" range_max="6.0"/>
-    <xacro:distance_sensor index="4" parent="tof_sensor_array_link" x="${r*cos((d_theta * 4) + phi)}" y="${r*sin((d_theta * 4) + phi)}" z="${-0.0175 / 2 + 0.025}" roll="0" pitch="${0}" yaw="${d_theta * 4 + phi}" range_min="0.001" range_max="6.0"/>
-    <xacro:distance_sensor index="5" parent="tof_sensor_array_link" x="${r*cos((d_theta * 5) + phi)}" y="${r*sin((d_theta * 5) + phi)}" z="${-0.0175 / 2 + 0.025}" roll="0" pitch="${0}" yaw="${d_theta * 5 + phi}" range_min="0.001" range_max="6.0"/>
-    <xacro:distance_sensor index="6" parent="tof_sensor_array_link" x="${r*cos((d_theta * 6) + phi)}" y="${r*sin((d_theta * 6) + phi)}" z="${-0.0175 / 2 + 0.025}" roll="0" pitch="${0}" yaw="${d_theta * 6 + phi}" range_min="0.001" range_max="6.0"/>
-    <xacro:distance_sensor index="7" parent="tof_sensor_array_link" x="${r*cos((d_theta * 7) + phi)}" y="${r*sin((d_theta * 7) + phi)}" z="${-0.0175 / 2 + 0.025}" roll="0" pitch="${0}" yaw="${d_theta * 7 + phi}" range_min="0.001" range_max="6.0"/>
+    <xacro:distance_sensor index="0" parent="tof_sensor_array_link" x="${r*cos((d_theta * 0) + phi)}" y="${r*sin((d_theta * 0) + phi)}" z="${0.03 / 2}" roll="0" pitch="${0}" yaw="${d_theta * 0 + phi}" range_min="0.001" range_max="6.0"/>
+    <xacro:distance_sensor index="1" parent="tof_sensor_array_link" x="${r*cos((d_theta * 1) + phi)}" y="${r*sin((d_theta * 1) + phi)}" z="${0.03 / 2}" roll="0" pitch="${0}" yaw="${d_theta * 1 + phi}" range_min="0.001" range_max="6.0"/>
+    <xacro:distance_sensor index="2" parent="tof_sensor_array_link" x="${r*cos((d_theta * 2) + phi)}" y="${r*sin((d_theta * 2) + phi)}" z="${0.03 / 2}" roll="0" pitch="${0}" yaw="${d_theta * 2 + phi}" range_min="0.001" range_max="6.0"/>
+    <xacro:distance_sensor index="3" parent="tof_sensor_array_link" x="${r*cos((d_theta * 3) + phi)}" y="${r*sin((d_theta * 3) + phi)}" z="${0.03 / 2}" roll="0" pitch="${0}" yaw="${d_theta * 3 + phi}" range_min="0.001" range_max="6.0"/>
+    <xacro:distance_sensor index="4" parent="tof_sensor_array_link" x="${r*cos((d_theta * 4) + phi)}" y="${r*sin((d_theta * 4) + phi)}" z="${0.03 / 2}" roll="0" pitch="${0}" yaw="${d_theta * 4 + phi}" range_min="0.001" range_max="6.0"/>
+    <xacro:distance_sensor index="5" parent="tof_sensor_array_link" x="${r*cos((d_theta * 5) + phi)}" y="${r*sin((d_theta * 5) + phi)}" z="${0.03 / 2}" roll="0" pitch="${0}" yaw="${d_theta * 5 + phi}" range_min="0.001" range_max="6.0"/>
+    <xacro:distance_sensor index="6" parent="tof_sensor_array_link" x="${r*cos((d_theta * 6) + phi)}" y="${r*sin((d_theta * 6) + phi)}" z="${0.03 / 2}" roll="0" pitch="${0}" yaw="${d_theta * 6 + phi}" range_min="0.001" range_max="6.0"/>
+    <xacro:distance_sensor index="7" parent="tof_sensor_array_link" x="${r*cos((d_theta * 7) + phi)}" y="${r*sin((d_theta * 7) + phi)}" z="${0.03 / 2}" roll="0" pitch="${0}" yaw="${d_theta * 7 + phi}" range_min="0.001" range_max="6.0"/>
     <xacro:distance_sensor index="8" parent="base_link" x="0" y="0" z="0.1" roll="0" pitch="${3 * pi / 2}" yaw="0" range_min="0.001" range_min_gazebo="0.015" range_max="6.0"/> <!-- up-facing sensor-->
-    <xacro:distance_sensor index="9" parent="tof_sensor_array_link" x="0" y="0" z="${0}" roll="0" pitch="${pi / 2}" yaw="0" range_min="0.001" range_min_gazebo="0.02" range_max="6.0"/> <!-- down-facing sensor -->
+    <xacro:distance_sensor index="9" parent="tof_sensor_array_link" x="0" y="0" z="${0}" roll="0" pitch="${pi / 2}" yaw="0" range_min="0.001" range_min_gazebo="0.001" range_max="6.0"/> <!-- down-facing sensor -->
   </xacro:if>
   <!-- Instantiate LED strip -->

File: clover_description/urdf/clover/clover4_macros.xacro (robot description, xacro)
@@ -153,5 +153,5 @@
     <xacro:property name="tof_sensor_drum_yaw_translate" value="${pi / 2 - pi / 8}" />
     <joint name="tof_sensor_array_joint" type="fixed">
-      <origin xyz="0 0 -0.07" rpy="0 0 ${tof_sensor_drum_yaw_translate}"/>
+      <origin xyz="0 0 -0.072" rpy="0 0 ${tof_sensor_drum_yaw_translate}"/>
       <parent link="base_link" />
       <child link="tof_sensor_array_link" />

Commit message: feat: simulation modifications to fix errors
* modified rpi cam translation
* added stiffness and dampening values to tof_sensor drum and sensor links
* removed unecessary remap of topic names

File: clover_description/urdf/clover/clover4.xacro (robot description, xacro)
@@ -13,5 +13,5 @@
   <!-- Create camera plugin -->
   <xacro:if value="$(arg main_camera)">
-    <xacro:property name="rpi_cam_x_translation" value="0.04" /> <!-- custom translation of rpi cam to make it -->
+    <xacro:property name="rpi_cam_x_translation" value="0.06" /> <!-- custom translation of rpi cam to make it -->
     <xacro:rpi_cam name="main_camera" parent="base_link" x="${0.055 + rpi_cam_x_translation}" y="0.0" z="-0.03" roll="0" pitch="${pi / 2}" yaw="0" width="320" height="240" rate="40" do_throttling="$(arg maintain_camera_rate)"/>
   </xacro:if>

File: clover_description/urdf/clover/clover4_macros.xacro (robot description, xacro)
@@ -62,5 +62,5 @@
            - sfalexrog
       -->
-      <collision>
+      <collision name="base_link_inertia_collision">
         <origin xyz="0 0 0" rpy="0 0 0" />
         <geometry>
@@ -69,4 +69,24 @@
       </collision>
     </link>
+    <gazebo reference="base_link">
+      <self_collide>0</self_collide>
+      <sensor name="base_link_contact" type="contact">
+        <always_on>true</always_on>
+        <contact>
+        <!-- See https://www.youtube.com/watch?v=KidqFt1mymE for why this
+             <collision> tag needs to be named differently than the actual
+             collision name it is referencing. The difference arises when `xacro`
+             is run to convert this file to sdf.
+             - simojo
+            -->
+          <collision>base_link_inertia_collision_collision</collision>
+        </contact>
+        <update_rate>5</update_rate>
+        <plugin name="base_link_bumper_plugin" filename="libgazebo_ros_bumper.so">
+          <bumperTopicName>base_link_contact</bumperTopicName>
+          <frameName>body</frameName>
+        </plugin>
+      </sensor>
+    </gazebo>
     <!-- This link is here for a single reason: to draw transparent parts (oh, and also to be the bane of my existence).
          I'm going to leave helpful comments for the poor soul who's going to attempt to improve this file.
@@ -162,4 +182,6 @@
     </gazebo>
     <gazebo reference="tof_sensor_array_link">
+      <kp>10000.0</kp>
+      <kd>10.0</kd>
       <material>flatblack</material> <!-- custom material. can be found in clover_description/media/materials/scripts/flatblack.material -->
     </gazebo>

File: clover_description/urdf/sensors/distance_sensor.urdf.xacro (robot description, xacro)
@@ -37,4 +37,6 @@
     <gazebo reference="${name}_${index}_link">
       <material>flatblack</material> <!-- custom material. can be found in clover_description/media/materials/scripts/flatblack.material -->
+      <kp>10000.0</kp>
+      <kd>10.0</kd>
       <sensor type="ray" name="${name}_${index}">
         <pose>0 0 0 0 0 0</pose>
