Commit message: feat: initializing tof_sensor_array_link

File: clover_description/urdf/clover/clover4_macros.xacro (robot description, xacro)
@@ -123,4 +123,45 @@
       <child link="base_guard_link" />
     </joint>
+    <!-- FIXME: how to set origin correctly? -->
+    <!-- FIXME: how to import assembly as a whole? -->
+    <!-- FIXME: how to add rangefinder sensors? -->
+    <link name="tof_sensor_array_link">
+      <inertial>
+        <!-- We give an oh-so-tiny mass to the link to avoid it being destroyed by Gazebo -->
+        <mass value="0.092"/> <!-- [kg] -->
+        <origin xyz="0 0 0" rpy="0 0 0"/>
+        <!-- We also give it some inertia, so that the physics engine does not go crazy
+             (and to avoid it being devoured by Gazebo)
+        -->
+        <!-- FIXME: calculate this -->
+        <inertia
+          ixx="${1/12 * 0.015 * 0.01 * 0.01}"
+          iyy="${1/12 * 0.015 * 0.01 * 0.01}"
+          izz="${1/12 * 0.015 * 0.01 * 0.01}"
+          ixy="0.0" ixz="0.0" iyz="0.0"
+        />
+      </inertial>
+      <!-- We may want to have proper collision tucked away here at some point, though -->
+      <collision>
+        <origin xyz="0 0 0" rpy="0 0 0" />
+        <geometry>
+          <box size="0.102 0.102 0.031" /> <!-- [m] [m] [m] -->
+        </geometry>
+      </collision>
+      <visual>
+        <!-- This origin should be the same as in "base_link_inertia" visuals -->
+        <origin xyz="0 0 0.025" rpy="0 0 0"/>
+        <geometry>
+          <mesh filename="package://clover_description/meshes/clover4/tof_sensor_array.base.dae"
+            scale="1 1 1"/>
+        </geometry>
+        <!-- Let me reiterate that you can't put the "material" tag to any effect -->
+      </visual>
+    </link>
+    <joint name="tof_sensor_array_joint" type="fixed">
+      <origin xyz="0 0 0" rpy="0 0 0"/>
+      <parent link="base_link" />
+      <child link="tof_sensor_array_link" />
+    </joint>
     <!-- attach multirotor_base_plugin to the base_link -->
     <gazebo>

Commit message: feat: inertial properties for tof_sensor_array

File: clover_description/urdf/clover/clover4_macros.xacro (robot description, xacro)
@@ -124,5 +124,4 @@
     </joint>
     <!-- FIXME: how to set origin correctly? -->
-    <!-- FIXME: how to import assembly as a whole? -->
     <!-- FIXME: how to add rangefinder sensors? -->
     <link name="tof_sensor_array_link">
@@ -134,10 +133,14 @@
              (and to avoid it being devoured by Gazebo)
         -->
-        <!-- FIXME: calculate this -->
         <inertia
-          ixx="${1/12 * 0.015 * 0.01 * 0.01}"
-          iyy="${1/12 * 0.015 * 0.01 * 0.01}"
-          izz="${1/12 * 0.015 * 0.01 * 0.01}"
-          ixy="0.0" ixz="0.0" iyz="0.0"
+          ixx="8.57890084602841e-5"
+          ixy="2.1174200194485434e-7"
+          ixz="4.585058826675158e-10"
+          iyx="2.1174200194485434e-7"
+          iyy="8.53655353895177e-5"
+          iyz="1.9573118871400868e-10"
+          izx="4.585058826675158e-10"
+          izy="1.9573118871400868e-10"
+          izz="0.0001459305357956103"
         />
       </inertial>
@@ -146,5 +149,5 @@
         <origin xyz="0 0 0" rpy="0 0 0" />
         <geometry>
-          <box size="0.102 0.102 0.031" /> <!-- [m] [m] [m] -->
+          <box size=".101567337 .101567337 .030500050" /> <!-- [m] [m] [m] -->
         </geometry>
       </collision>

Commit message: feat: scaling down sensor drum model

File: clover_description/urdf/clover/clover4_macros.xacro (robot description, xacro)
@@ -156,6 +156,6 @@
         <origin xyz="0 0 0.025" rpy="0 0 0"/>
         <geometry>
-          <mesh filename="package://clover_description/meshes/clover4/tof_sensor_array.base.dae"
-            scale="1 1 1"/>
+          <mesh filename="package://clover_description/meshes/clover4/tof_sensor_drum.dae"
+            scale="0.001 0.001 0.001"/> <!-- scale down because model is represented in mm -->
         </geometry>
         <!-- Let me reiterate that you can't put the "material" tag to any effect -->

Commit message: feat: clover_simulation: accomodating multiple ranging sensors

File: clover_description/urdf/clover/clover4_macros.xacro (robot description, xacro)
@@ -127,10 +127,6 @@
     <link name="tof_sensor_array_link">
       <inertial>
-        <!-- We give an oh-so-tiny mass to the link to avoid it being destroyed by Gazebo -->
         <mass value="0.092"/> <!-- [kg] -->
         <origin xyz="0 0 0" rpy="0 0 0"/>
-        <!-- We also give it some inertia, so that the physics engine does not go crazy
-             (and to avoid it being devoured by Gazebo)
-        -->
         <inertia
           ixx="8.57890084602841e-5"
@@ -145,5 +141,4 @@
         />
       </inertial>
-      <!-- We may want to have proper collision tucked away here at some point, though -->
       <collision>
         <origin xyz="0 0 0" rpy="0 0 0" />
@@ -153,5 +148,4 @@
       </collision>
       <visual>
-        <!-- This origin should be the same as in "base_link_inertia" visuals -->
         <origin xyz="0 0 0.025" rpy="0 0 0"/>
         <geometry>
@@ -159,5 +153,4 @@
             scale="0.001 0.001 0.001"/> <!-- scale down because model is represented in mm -->
         </geometry>
-        <!-- Let me reiterate that you can't put the "material" tag to any effect -->
       </visual>
     </link>
@@ -167,4 +160,11 @@
       <child link="tof_sensor_array_link" />
     </joint>
+    <gazebo reference="tof_sensor_array_joint">
+      <disableFixedJointLumping>true</disableFixedJointLumping>
+      <preserveFixedJoint>true</preserveFixedJoint>
+    </gazebo>
+    <gazebo reference="tof_sensor_array_link">
+      <material>Gazebo/FlatBlack</material>
+    </gazebo>
     <!-- attach multirotor_base_plugin to the base_link -->
     <gazebo>

Commit message: fix: scaling

File: clover_description/urdf/clover/clover4_macros.xacro (robot description, xacro)
@@ -128,5 +128,5 @@
       <inertial>
         <mass value="0.092"/> <!-- [kg] -->
-        <origin xyz="0 0 0" rpy="0 0 0"/>
+        <origin xyz="0 0 ${-1 * 0.01525 / 2}" rpy="0 0 0"/>
         <inertia
           ixx="8.57890084602841e-5"
@@ -151,5 +151,5 @@
         <geometry>
           <mesh filename="package://clover_description/meshes/clover4/tof_sensor_drum.dae"
-            scale="0.001 0.001 0.001"/> <!-- scale down because model is represented in mm -->
+            scale="0.01 0.01 0.01"/> <!-- scale down because model is represented in mm -->
         </geometry>
       </visual>

Commit message: feat: simulation speed, custom material

File: clover_description/urdf/clover/clover4_macros.xacro (robot description, xacro)
@@ -165,5 +165,5 @@
     </gazebo>
     <gazebo reference="tof_sensor_array_link">
-      <material>Gazebo/FlatBlack</material>
+      <material>flatblack</material> <!-- custom material. can be found in clover_description/media/materials/scripts/flatblack.material -->
     </gazebo>
     <!-- attach multirotor_base_plugin to the base_link -->

Commit message: feat: joint positioning

File: clover_description/urdf/clover/clover4_macros.xacro (robot description, xacro)
@@ -133,14 +133,11 @@
           ixy="2.1174200194485434e-7"
           ixz="4.585058826675158e-10"
-          iyx="2.1174200194485434e-7"
           iyy="8.53655353895177e-5"
           iyz="1.9573118871400868e-10"
-          izx="4.585058826675158e-10"
-          izy="1.9573118871400868e-10"
           izz="0.0001459305357956103"
         />
       </inertial>
       <collision>
-        <origin xyz="0 0 0" rpy="0 0 0" />
+        <origin xyz="0 0 -0.015" rpy="0 0 0" />
         <geometry>
           <box size=".101567337 .101567337 .030500050" /> <!-- [m] [m] [m] -->
@@ -148,5 +145,5 @@
       </collision>
       <visual>
-        <origin xyz="0 0 0.025" rpy="0 0 0"/>
+        <origin xyz="0 0 -0.015" rpy="0 0 0"/>
         <geometry>
           <mesh filename="package://clover_description/meshes/clover4/tof_sensor_drum.dae"
@@ -156,5 +153,5 @@
     </link>
     <joint name="tof_sensor_array_joint" type="fixed">
-      <origin xyz="0 0 0" rpy="0 0 0"/>
+      <origin xyz="0 0 -0.015" rpy="0 0 0"/>
       <parent link="base_link" />
       <child link="tof_sensor_array_link" />

Commit message: feat/wip: adding leg links to mock real-life clover model

File: clover_description/urdf/clover/clover4_macros.xacro (robot description, xacro)
@@ -143,9 +143,177 @@
       <child link="base_guard_link" />
     </joint>
+    <xacro:property name="base_leg_x_dimension" value="0.045" />
+    <xacro:property name="base_leg_y_dimension" value="0.007" />
+    <xacro:property name="base_leg_z_dimension" value="0.15" />
+    <xacro:property name="base_leg_mass" value="0.001" />
+    <xacro:property name="base_leg_r" value="0.1" /> <!-- radius of base_leg joint origin from quadcopter center of mass -->
+    <xacro:property name="base_leg_theta" value="${pi / 2}" /> <!-- angle to increment base_leg yaw around quadcopter frame -->
+    <xacro:property name="base_leg_phi" value="${pi / 4}" /> <!-- angle offset to start from -->
+    <joint name="base_leg_1_joint" type="fixed">
+      <origin xyz="${cos(0 * base_leg_theta + base_leg_phi) * base_leg_r} ${sin(0 * base_leg_theta + base_leg_phi) * base_leg_r} 0" rpy="0 0 ${0 * base_leg_theta + base_leg_phi}" />
+      <parent link="base_link" />
+      <child link="base_leg_1" />
+    </joint>
+    <gazebo reference="base_leg_1_joint">
+      <disableFixedJointLumping>true</disableFixedJointLumping>
+      <preserveFixedJoint>true</preserveFixedJoint>
+    </gazebo>
+    <joint name="base_leg_2_joint" type="fixed">
+      <origin xyz="${cos(1 * base_leg_theta + base_leg_phi) * base_leg_r} ${sin(1 * base_leg_theta + base_leg_phi) * base_leg_r} 0" rpy="0 0 ${1 * base_leg_theta + base_leg_phi}" />
+      <parent link="base_link" />
+      <child link="base_leg_2" />
+    </joint>
+    <gazebo reference="base_leg_2_joint">
+      <disableFixedJointLumping>true</disableFixedJointLumping>
+      <preserveFixedJoint>true</preserveFixedJoint>
+    </gazebo>
+    <joint name="base_leg_3_joint" type="fixed">
+      <origin xyz="${cos(2 * base_leg_theta + base_leg_phi) * base_leg_r} ${sin(2 * base_leg_theta + base_leg_phi) * base_leg_r} 0" rpy="0 0 ${2 * base_leg_theta + base_leg_phi}" />
+      <parent link="base_link" />
+      <child link="base_leg_3" />
+    </joint>
+    <gazebo reference="base_leg_3_joint">
+      <disableFixedJointLumping>true</disableFixedJointLumping>
+      <preserveFixedJoint>true</preserveFixedJoint>
+    </gazebo>
+    <joint name="base_leg_4_joint" type="fixed">
+      <origin xyz="${cos(3 * base_leg_theta + base_leg_phi) * base_leg_r} ${sin(3 * base_leg_theta + base_leg_phi) * base_leg_r} 0" rpy="0 0 ${3 * base_leg_theta + base_leg_phi}" />
+      <parent link="base_link" />
+      <child link="base_leg_4" />
+    </joint>
+    <gazebo reference="base_leg_4_joint">
+      <disableFixedJointLumping>true</disableFixedJointLumping>
+      <preserveFixedJoint>true</preserveFixedJoint>
+    </gazebo>
+    <link name="base_leg_1">
+      <inertial>
+        <mass value="${base_leg_mass}"/> <!-- [kg] -->
+        <origin xyz="0 0 ${-1 * base_leg_z_dimension / 2}" rpy="0 0 0"/>
+        <inertia
+          ixx="${1/12 * base_leg_mass * (base_leg_y_dimension * base_leg_y_dimension + base_leg_z_dimension * base_leg_z_dimension)}"
+          ixy="0.0"
+          ixz="0.0"
+          iyy="${1/12 * base_leg_mass * (base_leg_x_dimension * base_leg_x_dimension + base_leg_z_dimension * base_leg_z_dimension)}"
+          iyz="0.0"
+          izz="${1/12 * base_leg_mass * (base_leg_x_dimension * base_leg_x_dimension + base_leg_y_dimension * base_leg_y_dimension)}"
+        />
+      </inertial>
+      <collision>
+        <origin xyz="0 0 ${-1 * base_leg_z_dimension / 2}" rpy="0 0 0"/>
+        <geometry>
+          <box size="${base_leg_x_dimension} ${base_leg_y_dimension} ${base_leg_z_dimension}" /> <!-- [m] [m] [m] -->
+        </geometry>
+      </collision>
+      <visual>
+        <origin xyz="0 0 ${-1 * base_leg_z_dimension / 2}" rpy="0 0 0"/>
+        <geometry>
+          <box size="${base_leg_x_dimension} ${base_leg_y_dimension} ${base_leg_z_dimension}" /> <!-- [m] [m] [m] -->
+        </geometry>
+      </visual>
+    </link>
+    <gazebo reference="base_leg_1">
+      <!-- <kp>10000.0</kp> -->
+      <!-- <kd>10.0</kd> -->
+      <material>Polycarbonate</material> <!-- custom material. can be found in clover_description/media/materials/ -->
+    </gazebo>
+    <link name="base_leg_2">
+      <inertial>
+        <mass value="${base_leg_mass}"/> <!-- [kg] -->
+        <origin xyz="0 0 ${-1 * base_leg_z_dimension / 2}" rpy="0 0 0"/>
+        <inertia
+          ixx="${1/12 * base_leg_mass * (base_leg_y_dimension * base_leg_y_dimension + base_leg_z_dimension * base_leg_z_dimension)}"
+          ixy="0.0"
+          ixz="0.0"
+          iyy="${1/12 * base_leg_mass * (base_leg_x_dimension * base_leg_x_dimension + base_leg_z_dimension * base_leg_z_dimension)}"
+          iyz="0.0"
+          izz="${1/12 * base_leg_mass * (base_leg_x_dimension * base_leg_x_dimension + base_leg_y_dimension * base_leg_y_dimension)}"
+        />
+      </inertial>
+      <collision>
+        <origin xyz="0 0 ${-1 * base_leg_z_dimension / 2}" rpy="0 0 0"/>
+        <geometry>
+          <box size="${base_leg_x_dimension} ${base_leg_y_dimension} ${base_leg_z_dimension}" /> <!-- [m] [m] [m] -->
+        </geometry>
+      </collision>
+      <visual>
+        <origin xyz="0 0 ${-1 * base_leg_z_dimension / 2}" rpy="0 0 0"/>
+        <geometry>
+          <box size="${base_leg_x_dimension} ${base_leg_y_dimension} ${base_leg_z_dimension}" /> <!-- [m] [m] [m] -->
+        </geometry>
+      </visual>
+    </link>
+    <gazebo reference="base_leg_2">
+      <!-- <kp>10000.0</kp> -->
+      <!-- <kd>10.0</kd> -->
+      <material>Polycarbonate</material> <!-- custom material. can be found in clover_description/media/materials/ -->
+    </gazebo>
+    <link name="base_leg_3">
+      <inertial>
+        <mass value="${base_leg_mass}"/> <!-- [kg] -->
+        <origin xyz="0 0 ${-1 * base_leg_z_dimension / 2}" rpy="0 0 0"/>
+        <inertia
+          ixx="${1/12 * base_leg_mass * (base_leg_y_dimension * base_leg_y_dimension + base_leg_z_dimension * base_leg_z_dimension)}"
+          ixy="0.0"
+          ixz="0.0"
+          iyy="${1/12 * base_leg_mass * (base_leg_x_dimension * base_leg_x_dimension + base_leg_z_dimension * base_leg_z_dimension)}"
+          iyz="0.0"
+          izz="${1/12 * base_leg_mass * (base_leg_x_dimension * base_leg_x_dimension + base_leg_y_dimension * base_leg_y_dimension)}"
+        />
+      </inertial>
+      <collision>
+        <origin xyz="0 0 ${-1 * base_leg_z_dimension / 2}" rpy="0 0 0"/>
+        <geometry>
+          <box size="${base_leg_x_dimension} ${base_leg_y_dimension} ${base_leg_z_dimension}" /> <!-- [m] [m] [m] -->
+        </geometry>
+      </collision>
+      <visual>
+        <origin xyz="0 0 ${-1 * base_leg_z_dimension / 2}" rpy="0 0 0"/>
+        <geometry>
+          <box size="${base_leg_x_dimension} ${base_leg_y_dimension} ${base_leg_z_dimension}" /> <!-- [m] [m] [m] -->
+        </geometry>
+      </visual>
+    </link>
+    <gazebo reference="base_leg_3">
+      <!-- <kp>10000.0</kp> -->
+      <!-- <kd>10.0</kd> -->
+      <material>Polycarbonate</material> <!-- custom material. can be found in clover_description/media/materials/ -->
+    </gazebo>
+    <link name="base_leg_4">
+      <inertial>
+        <mass value="${base_leg_mass}"/> <!-- [kg] -->
+        <origin xyz="0 0 ${-1 * base_leg_z_dimension / 2}" rpy="0 0 0"/>
+        <!-- reference: https://en.wikipedia.org/wiki/List_of_moments_of_inertia (see solid cuboid) -->
+        <inertia
+          ixx="${1/12 * base_leg_mass * (base_leg_y_dimension * base_leg_y_dimension + base_leg_z_dimension * base_leg_z_dimension)}"
+          ixy="0.0"
+          ixz="0.0"
+          iyy="${1/12 * base_leg_mass * (base_leg_x_dimension * base_leg_x_dimension + base_leg_z_dimension * base_leg_z_dimension)}"
+          iyz="0.0"
+          izz="${1/12 * base_leg_mass * (base_leg_x_dimension * base_leg_x_dimension + base_leg_y_dimension * base_leg_y_dimension)}"
+        />
+      </inertial>
+      <collision>
+        <origin xyz="0 0 ${-1 * base_leg_z_dimension / 2}" rpy="0 0 0"/>
+        <geometry>
+          <box size="${base_leg_x_dimension} ${base_leg_y_dimension} ${base_leg_z_dimension}" /> <!-- [m] [m] [m] -->
+        </geometry>
+      </collision>
+      <visual>
+        <origin xyz="0 0 ${-1 * base_leg_z_dimension / 2}" rpy="0 0 0"/>
+        <geometry>
+          <box size="${base_leg_x_dimension} ${base_leg_y_dimension} ${base_leg_z_dimension}" /> <!-- [m] [m] [m] -->
+        </geometry>
+      </visual>
+    </link>
+    <gazebo reference="base_leg_4">
+      <!-- <kp>10000.0</kp> -->
+      <!-- <kd>10.0</kd> -->
+      <material>Polycarbonate</material> <!-- custom material. can be found in clover_description/media/materials/ -->
+    </gazebo>
     <!-- FIXME: how to set origin correctly? -->
     <link name="tof_sensor_array_link">
       <inertial>
         <mass value="0.092"/> <!-- [kg] -->
-        <origin xyz="0 0 0" rpy="0 0 0"/>
+        <origin xyz="0 0 0" rpy="0 0 0" />
         <inertia
           ixx="8.57890084602841e-5"
@@ -164,5 +332,5 @@
       </collision>
       <visual>
-        <origin xyz="0 0 0" rpy="0 0 0"/>
+        <origin xyz="0 0 0" rpy="0 0 0" />
         <geometry>
           <mesh filename="package://clover_description/meshes/clover4/tof_sensor_drum.dae"

Commit message: feat: adding damping values to legs, untranslating parquet plane, and reducing collision box size of body

File: clover_description/urdf/clover/clover4_macros.xacro (robot description, xacro)
@@ -63,5 +63,5 @@
       -->
       <collision name="base_link_inertia_collision">
-        <origin xyz="0 0 0" rpy="0 0 0" />
+        <origin xyz="0 0 0.05" rpy="0 0 0" />
         <geometry>
           <box size="${body_width} ${body_width} ${body_height}" /> <!-- [m] [m] [m] -->
@@ -213,6 +213,6 @@
     </link>
     <gazebo reference="base_leg_1">
-      <!-- <kp>10000.0</kp> -->
-      <!-- <kd>10.0</kd> -->
+      <kp>10000.0</kp>
+      <kd>10.0</kd>
       <material>Polycarbonate</material> <!-- custom material. can be found in clover_description/media/materials/ -->
     </gazebo>
@@ -244,6 +244,6 @@
     </link>
     <gazebo reference="base_leg_2">
-      <!-- <kp>10000.0</kp> -->
-      <!-- <kd>10.0</kd> -->
+      <kp>10000.0</kp>
+      <kd>10.0</kd>
       <material>Polycarbonate</material> <!-- custom material. can be found in clover_description/media/materials/ -->
     </gazebo>
@@ -275,6 +275,6 @@
     </link>
     <gazebo reference="base_leg_3">
-      <!-- <kp>10000.0</kp> -->
-      <!-- <kd>10.0</kd> -->
+      <kp>10000.0</kp>
+      <kd>10.0</kd>
       <material>Polycarbonate</material> <!-- custom material. can be found in clover_description/media/materials/ -->
     </gazebo>
@@ -307,6 +307,6 @@
     </link>
     <gazebo reference="base_leg_4">
-      <!-- <kp>10000.0</kp> -->
-      <!-- <kd>10.0</kd> -->
+      <kp>10000.0</kp>
+      <kd>10.0</kd>
       <material>Polycarbonate</material> <!-- custom material. can be found in clover_description/media/materials/ -->
     </gazebo>

File: clover_description/urdf/clover/clover4_physics.xacro (robot description, xacro)
@@ -15,5 +15,5 @@
   </xacro:unless>
   <xacro:property name="body_width" value="0.35" /> <!-- [m] -->
-  <xacro:property name="body_height" value="0.124" /> <!-- [m] -->
+  <xacro:property name="body_height" value="0.10" /> <!-- [m] -->
   <xacro:property name="mass_rotor" value="0.01" /> <!-- [kg] -->
   <xacro:property name="arm_length_front_x" value="0.083" /> <!-- [m] -->
