Commit message: feat: modularizing base_leg model, and fixing issue with wiggly legs

File: clover_description/urdf/clover/clover4_macros.xacro (robot description, xacro)
@@ -143,172 +143,4 @@
       <child link="base_guard_link" />
     </joint>
-    <xacro:property name="base_leg_x_dimension" value="0.045" />
-    <xacro:property name="base_leg_y_dimension" value="0.007" />
-    <xacro:property name="base_leg_z_dimension" value="0.15" />
-    <xacro:property name="base_leg_mass" value="0.001" />
-    <xacro:property name="base_leg_r" value="0.1" /> <!-- radius of base_leg joint origin from quadcopter center of mass -->
-    <xacro:property name="base_leg_theta" value="${pi / 2}" /> <!-- angle to increment base_leg yaw around quadcopter frame -->
-    <xacro:property name="base_leg_phi" value="${pi / 4}" /> <!-- angle offset to start from -->
-    <joint name="base_leg_1_joint" type="fixed">
-      <origin xyz="${cos(0 * base_leg_theta + base_leg_phi) * base_leg_r} ${sin(0 * base_leg_theta + base_leg_phi) * base_leg_r} 0" rpy="0 0 ${0 * base_leg_theta + base_leg_phi}" />
-      <parent link="base_link" />
-      <child link="base_leg_1" />
-    </joint>
-    <gazebo reference="base_leg_1_joint">
-      <disableFixedJointLumping>true</disableFixedJointLumping>
-      <preserveFixedJoint>true</preserveFixedJoint>
-    </gazebo>
-    <joint name="base_leg_2_joint" type="fixed">
-      <origin xyz="${cos(1 * base_leg_theta + base_leg_phi) * base_leg_r} ${sin(1 * base_leg_theta + base_leg_phi) * base_leg_r} 0" rpy="0 0 ${1 * base_leg_theta + base_leg_phi}" />
-      <parent link="base_link" />
-      <child link="base_leg_2" />
-    </joint>
-    <gazebo reference="base_leg_2_joint">
-      <disableFixedJointLumping>true</disableFixedJointLumping>
-      <preserveFixedJoint>true</preserveFixedJoint>
-    </gazebo>
-    <joint name="base_leg_3_joint" type="fixed">
-      <origin xyz="${cos(2 * base_leg_theta + base_leg_phi) * base_leg_r} ${sin(2 * base_leg_theta + base_leg_phi) * base_leg_r} 0" rpy="0 0 ${2 * base_leg_theta + base_leg_phi}" />
-      <parent link="base_link" />
-      <child link="base_leg_3" />
-    </joint>
-    <gazebo reference="base_leg_3_joint">
-      <disableFixedJointLumping>true</disableFixedJointLumping>
-      <preserveFixedJoint>true</preserveFixedJoint>
-    </gazebo>
-    <joint name="base_leg_4_joint" type="fixed">
-      <origin xyz="${cos(3 * base_leg_theta + base_leg_phi) * base_leg_r} ${sin(3 * base_leg_theta + base_leg_phi) * base_leg_r} 0" rpy="0 0 ${3 * base_leg_theta + base_leg_phi}" />
-      <parent link="base_link" />
-      <child link="base_leg_4" />
-    </joint>
-    <gazebo reference="base_leg_4_joint">
-      <disableFixedJointLumping>true</disableFixedJointLumping>
-      <preserveFixedJoint>true</preserveFixedJoint>
-    </gazebo>
-    <link name="base_leg_1">
-      <inertial>
-        <mass value="${base_leg_mass}"/> <!-- [kg] -->
-        <origin xyz="0 0 ${-1 * base_leg_z_dimension / 2}" rpy="0 0 0"/>
-        <inertia
-          ixx="${1/12 * base_leg_mass * (base_leg_y_dimension * base_leg_y_dimension + base_leg_z_dimension * base_leg_z_dimension)}"
-          ixy="0.0"
-          ixz="0.0"
-          iyy="${1/12 * base_leg_mass * (base_leg_x_dimension * base_leg_x_dimension + base_leg_z_dimension * base_leg_z_dimension)}"
-          iyz="0.0"
-          izz="${1/12 * base_leg_mass * (base_leg_x_dimension * base_leg_x_dimension + base_leg_y_dimension * base_leg_y_dimension)}"
-        />
-      </inertial>
-      <collision>
-        <origin xyz="0 0 ${-1 * base_leg_z_dimension / 2}" rpy="0 0 0"/>
-        <geometry>
-          <box size="${base_leg_x_dimension} ${base_leg_y_dimension} ${base_leg_z_dimension}" /> <!-- [m] [m] [m] -->
-        </geometry>
-      </collision>
-      <visual>
-        <origin xyz="0 0 ${-1 * base_leg_z_dimension / 2}" rpy="0 0 0"/>
-        <geometry>
-          <box size="${base_leg_x_dimension} ${base_leg_y_dimension} ${base_leg_z_dimension}" /> <!-- [m] [m] [m] -->
-        </geometry>
-      </visual>
-    </link>
-    <gazebo reference="base_leg_1">
-      <kp>10000.0</kp>
-      <kd>10.0</kd>
-      <material>Polycarbonate</material> <!-- custom material. can be found in clover_description/media/materials/ -->
-    </gazebo>
-    <link name="base_leg_2">
-      <inertial>
-        <mass value="${base_leg_mass}"/> <!-- [kg] -->
-        <origin xyz="0 0 ${-1 * base_leg_z_dimension / 2}" rpy="0 0 0"/>
-        <inertia
-          ixx="${1/12 * base_leg_mass * (base_leg_y_dimension * base_leg_y_dimension + base_leg_z_dimension * base_leg_z_dimension)}"
-          ixy="0.0"
-          ixz="0.0"
-          iyy="${1/12 * base_leg_mass * (base_leg_x_dimension * base_leg_x_dimension + base_leg_z_dimension * base_leg_z_dimension)}"
-          iyz="0.0"
-          izz="${1/12 * base_leg_mass * (base_leg_x_dimension * base_leg_x_dimension + base_leg_y_dimension * base_leg_y_dimension)}"
-        />
-      </inertial>
-      <collision>
-        <origin xyz="0 0 ${-1 * base_leg_z_dimension / 2}" rpy="0 0 0"/>
-        <geometry>
-          <box size="${base_leg_x_dimension} ${base_leg_y_dimension} ${base_leg_z_dimension}" /> <!-- [m] [m] [m] -->
-        </geometry>
-      </collision>
-      <visual>
-        <origin xyz="0 0 ${-1 * base_leg_z_dimension / 2}" rpy="0 0 0"/>
-        <geometry>
-          <box size="${base_leg_x_dimension} ${base_leg_y_dimension} ${base_leg_z_dimension}" /> <!-- [m] [m] [m] -->
-        </geometry>
-      </visual>
-    </link>
-    <gazebo reference="base_leg_2">
-      <kp>10000.0</kp>
-      <kd>10.0</kd>
-      <material>Polycarbonate</material> <!-- custom material. can be found in clover_description/media/materials/ -->
-    </gazebo>
-    <link name="base_leg_3">
-      <inertial>
-        <mass value="${base_leg_mass}"/> <!-- [kg] -->
-        <origin xyz="0 0 ${-1 * base_leg_z_dimension / 2}" rpy="0 0 0"/>
-        <inertia
-          ixx="${1/12 * base_leg_mass * (base_leg_y_dimension * base_leg_y_dimension + base_leg_z_dimension * base_leg_z_dimension)}"
-          ixy="0.0"
-          ixz="0.0"
-          iyy="${1/12 * base_leg_mass * (base_leg_x_dimension * base_leg_x_dimension + base_leg_z_dimension * base_leg_z_dimension)}"
-          iyz="0.0"
-          izz="${1/12 * base_leg_mass * (base_leg_x_dimension * base_leg_x_dimension + base_leg_y_dimension * base_leg_y_dimension)}"
-        />
-      </inertial>
-      <collision>
-        <origin xyz="0 0 ${-1 * base_leg_z_dimension / 2}" rpy="0 0 0"/>
-        <geometry>
-          <box size="${base_leg_x_dimension} ${base_leg_y_dimension} ${base_leg_z_dimension}" /> <!-- [m] [m] [m] -->
-        </geometry>
-      </collision>
-      <visual>
-        <origin xyz="0 0 ${-1 * base_leg_z_dimension / 2}" rpy="0 0 0"/>
-        <geometry>
-          <box size="${base_leg_x_dimension} ${base_leg_y_dimension} ${base_leg_z_dimension}" /> <!-- [m] [m] [m] -->
-        </geometry>
-      </visual>
-    </link>
-    <gazebo reference="base_leg_3">
-      <kp>10000.0</kp>
-      <kd>10.0</kd>
-      <material>Polycarbonate</material> <!-- custom material. can be found in clover_description/media/materials/ -->
-    </gazebo>
-    <link name="base_leg_4">
-      <inertial>
-        <mass value="${base_leg_mass}"/> <!-- [kg] -->
-        <origin xyz="0 0 ${-1 * base_leg_z_dimension / 2}" rpy="0 0 0"/>
-        <!-- reference: https://en.wikipedia.org/wiki/List_of_moments_of_inertia (see solid cuboid) -->
-        <inertia
-          ixx="${1/12 * base_leg_mass * (base_leg_y_dimension * base_leg_y_dimension + base_leg_z_dimension * base_leg_z_dimension)}"
-          ixy="0.0"
-          ixz="0.0"
-          iyy="${1/12 * base_leg_mass * (base_leg_x_dimension * base_leg_x_dimension + base_leg_z_dimension * base_leg_z_dimension)}"
-          iyz="0.0"
-          izz="${1/12 * base_leg_mass * (base_leg_x_dimension * base_leg_x_dimension + base_leg_y_dimension * base_leg_y_dimension)}"
-        />
-      </inertial>
-      <collision>
-        <origin xyz="0 0 ${-1 * base_leg_z_dimension / 2}" rpy="0 0 0"/>
-        <geometry>
-          <box size="${base_leg_x_dimension} ${base_leg_y_dimension} ${base_leg_z_dimension}" /> <!-- [m] [m] [m] -->
-        </geometry>
-      </collision>
-      <visual>
-        <origin xyz="0 0 ${-1 * base_leg_z_dimension / 2}" rpy="0 0 0"/>
-        <geometry>
-          <box size="${base_leg_x_dimension} ${base_leg_y_dimension} ${base_leg_z_dimension}" /> <!-- [m] [m] [m] -->
-        </geometry>
-      </visual>
-    </link>
-    <gazebo reference="base_leg_4">
-      <kp>10000.0</kp>
-      <kd>10.0</kd>
-      <material>Polycarbonate</material> <!-- custom material. can be found in clover_description/media/materials/ -->
-    </gazebo>
     <!-- FIXME: how to set origin correctly? -->
     <link name="tof_sensor_array_link">
@@ -326,5 +158,5 @@
       </inertial>
       <collision>
-        <origin xyz="0 0 0" rpy="0 0 0" />
+        <origin xyz="0 0 ${.030500050 / 2}" rpy="0 0 0" />
         <geometry>
           <box size=".101567337 .101567337 .030500050" /> <!-- [m] [m] [m] -->

File: clover_description/urdf/clover/clover4_physics.xacro (robot description, xacro)
@@ -88,4 +88,11 @@
     <xacro:insert_block name="body_inertia" />
   </xacro:clover4_base_macro>
+  <!-- Included URDF Files -->
+  <xacro:include filename="clover4_base_leg.xacro" />
+  <!-- Instantiate leg models -->
+  <xacro:clover4_base_leg parent="base_link" index="0" />
+  <xacro:clover4_base_leg parent="base_link" index="1" />
+  <xacro:clover4_base_leg parent="base_link" index="2" />
+  <xacro:clover4_base_leg parent="base_link" index="3" />
   <!-- Instantiate rotors -->
   <xacro:vertical_clover_rotor
