Commit message: feat: adding option to make clover legs transparent to avoid interference with camera

File: clover_description/urdf/clover/clover4_base_leg.xacro (robot description, xacro)
@@ -6,5 +6,5 @@
 <robot xmlns:xacro="http://ros.org/wiki/xacro">
   <xacro:macro name="clover4_base_leg"
-    params="parent:=base_link index">
+    params="parent:=base_link index transparent:=false">
     <xacro:property name="base_leg_x_dimension" value="0.045" />
     <xacro:property name="base_leg_y_dimension" value="0.007" />
@@ -39,10 +39,12 @@
         </geometry>
       </collision>
-      <visual>
-        <origin xyz="0 0 ${-1 * base_leg_z_dimension / 2}" rpy="0 0 0"/>
-        <geometry>
-          <box size="${base_leg_x_dimension} ${base_leg_y_dimension} ${base_leg_z_dimension}" /> <!-- [m] [m] [m] -->
-        </geometry>
-      </visual>
+      <xacro:unless value="${transparent}">
+        <visual>
+          <origin xyz="0 0 ${-1 * base_leg_z_dimension / 2}" rpy="0 0 0"/>
+          <geometry>
+            <box size="${base_leg_x_dimension} ${base_leg_y_dimension} ${base_leg_z_dimension}" /> <!-- [m] [m] [m] -->
+          </geometry>
+        </visual>
+      </xacro:unless>
     </link>
     <!--

File: clover_description/urdf/clover/clover4_physics.xacro (robot description, xacro)
@@ -91,8 +91,8 @@
   <xacro:include filename="clover4_base_leg.xacro" />
   <!-- Instantiate leg models -->
-  <xacro:clover4_base_leg parent="base_link" index="0" />
-  <xacro:clover4_base_leg parent="base_link" index="1" />
-  <xacro:clover4_base_leg parent="base_link" index="2" />
-  <xacro:clover4_base_leg parent="base_link" index="3" />
+  <xacro:clover4_base_leg parent="base_link" index="0" transparent="true" /> <!-- set to transparent to not interfere with camera -->
+  <xacro:clover4_base_leg parent="base_link" index="1" transparent="false" />
+  <xacro:clover4_base_leg parent="base_link" index="2" transparent="false" />
+  <xacro:clover4_base_leg parent="base_link" index="3" transparent="true" /> <!-- set to transparent to not interfere with camera -->
   <!-- Instantiate rotors -->
   <xacro:vertical_clover_rotor
